File: KiCAD/Z80-1MSRAM.sch (KiCad schematic (older format))
At the start: 24 parts, among them J1 SBC8080 BUS, U1 7402, U2 74HC573, U3 74HC139, U4 74HC04, U5 74HC00, U6 628128, U7 28C256

Commit message: REV2基板対応
Parts:
- removed U2: 74HC573, Housings_DIP:DIP-20_W7.62mm_Socket, symbol Z80-1MSRAM-rescue:74LS573
- added D3: LED, LED_THT:LED_D3.0mm, symbol Device:LED
- added J2: I/O ADDR SEL, Connector_PinHeader_2.54mm:PinHeader_2x04_P2.54mm_Vertical, symbol Connector_Generic:Conn_02x04_Odd_Even
- added R3: 1k, Resistor_THT:R_Axial_DIN0207_L6.3mm_D2.5mm_P10.16mm_Horizontal, symbol Device:R
- added U2: 74HC74, Package_DIP:DIP-14_W7.62mm_Socket, symbol 74xx:74HC74
- U1: value 7402 -> 74HC02
Connections:
- net labels added: RES
- net labels removed: ~MSEL
- wire segments 222 -> 255
- no-connect marks 26 -> 13
Other:
- note removed: "IO ADDR : 80H"
- moved on the sheet: C1, C2, C3, C4, C5, C6, C7, C8, D1, D2, R1, R2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

Commit message: REV3 基板関係 試作バージョン
Parts:
- added JP1: A7_Jumper, Connector_PinHeader_2.54mm:PinHeader_1x03_P2.54mm_Vertical, symbol Jumper:Jumper_3_Open
- added Q1: 2SC1815, Package_TO_SOT_THT:TO-92L_Inline_Wide, symbol Transistor_BJT:2SC1815
- added R4: 100k, Resistor_THT:R_Axial_DIN0207_L6.3mm_D2.5mm_P10.16mm_Horizontal, symbol Device:R_US
- added R5: 1k, Resistor_THT:R_Axial_DIN0207_L6.3mm_D2.5mm_P10.16mm_Horizontal, symbol Device:R_US
- R1, R2: footprint Resistors_THT:R_Axial_DIN0207_L6.3mm_D2.5mm_P10.16mm_Horizontal -> Resistor_THT:R_Axial_DIN0207_L6.3mm_D2.5mm_P10.16mm_Horizontal
Connections:
- net A5: now also U3.2 (A0)
- net A6: now also U3.3 (A1); no longer U3.2 (A0)
- net A7: now also JP1.3 (B), R4.2; no longer U3.3 (A1)
- net GND: now also Q1.1 (E); no longer U3.1 (E)
- net VCC: now also R5.2
- new net: Q1.3 (B), R4.1
- new net: JP1.1 (A), Q1.2 (C), R5.1
- new net ADDR_SEL: JP1.2 (C), U3.1 (E)
Other:
- note added: "0xh-6xh"
- note added: "8xh-Exh"
Changed lines of the file:
@@
 Entry Bus Bus
 	8200 2600 8300 2700
-$Comp
-L Z80-1MSRAM-rescue:GND #PWR01
-U 1 1 5B6AD801
-P 5000 3850
-F 0 "#PWR01" H 5000 3600 50  0001 C CNN
-F 1 "GND" H 5000 3700 50  0000 C CNN
-F 2 "" H 5000 3850 50  0001 C CNN
-F 3 "" H 5000 3850 50  0001 C CNN
-	1    5000 3850
-	1    0    0    -1
-$EndComp
 Entry Wire Line
 	4850 3100 4950 3200
@@
 	4750 2600 4850 2700
 Text Label 5000 3200 0    60   ~ 0
-A7
+A6
 Text Label 5000 3350 0    60   ~ 0
-A6
+A5
 Entry Bus Bus
 	4200 2200 4300 2300
@@
 F 0 "R1" V 9980 7900 50  0000 C CNN
 F 1 "1k" V 9900 7900 50  0000 C CNN
-F 2 "Resistors_THT:R_Axial_DIN0207_L6.3mm_D2.5mm_P10.16mm_Horizontal" V 9830 7900 50  0001 C CNN
+F 2 "Resistor_THT:R_Axial_DIN0207_L6.3mm_D2.5mm_P10.16mm_Horizontal" V 9830 7900 50  0001 C CNN
 F 3 "" H 9900 7900 50  0001 C CNN
 	1    9900 7900
@@
 F 0 "R2" V 9980 8250 50  0000 C CNN
 F 1 "1k" V 9900 8250 50  0000 C CNN
-F 2 "Resistors_THT:R_Axial_DIN0207_L6.3mm_D2.5mm_P10.16mm_Horizontal" V 9830 8250 50  0001 C CNN
+F 2 "Resistor_THT:R_Axial_DIN0207_L6.3mm_D2.5mm_P10.16mm_Horizontal" V 9830 8250 50  0001 C CNN
 F 3 "" H 9900 8250 50  0001 C CNN
 	1    9900 8250
@@
 $EndComp
 Wire Wire Line
-	5000 3700 5000 3850
-Wire Wire Line
-	5200 3700 5000 3700
-Wire Wire Line
 	5200 3200 4950 3200
 Wire Wire Line
@@
 Wire Wire Line
 	2000 4400 2550 4400
+$Comp
+L Device:R_US R4
+U 1 1 5C8B2A5C
+P 4000 6250
+F 0 "R4" V 3900 6250 50  0000 C CNN
+F 1 "100k" V 4100 6250 50  0000 C CNN
+F 2 "Resistor_THT:R_Axial_DIN0207_L6.3mm_D2.5mm_P10.16mm_Horizontal" V 4040 6240 50  0001 C CNN
+F 3 "~" H 4000 6250 50  0001 C CNN
+	1    4000 6250
+	0    1    1    0
+$EndComp
+Text GLabel 3500 6250 0    60   Input ~ 0
+A7
+Wire Wire Line
+	3500 6250 3850 6250
+Wire Wire Line
+	4900 3700 5200 3700
+Text GLabel 4900 3700 0    60   Input ~ 0
+ADDR_SEL
+Text GLabel 5500 6350 2    60   Input ~ 0
+ADDR_SEL
+$Comp
+L Transistor_BJT:2SC1815 Q1
+U 1 1 5C8F8440
+P 4500 6250
+F 0 "Q1" H 4691 6296 50  0000 L CNN
+F 1 "2SC1815" H 4691 6205 50  0000 L CNN
+F 2 "Package_TO_SOT_THT:TO-92L_Inline_Wide" H 4700 6175 50  0001 L CIN
+F 3 "https://media.digikey.com/pdf/Data%20Sheets/Toshiba%20PDFs/2SC1815.pdf" H 4500 6250 50  0001 L CNN
+	1    4500 6250
+	1    0    0    -1
+$EndComp
+Wire Wire Line
+	4150 6250 4300 6250
+$Comp
+L Device:R_US R5
+U 1 1 5C90FB06
+P 4600 5800
+F 0 "R5" V 4500 5800 50  0000 C CNN
+F 1 "1k" V 4700 5800 50  0000 C CNN
+F 2 "Resistor_THT:R_Axial_DIN0207_L6.3mm_D2.5mm_P10.16mm_Horizontal" V 4640 5790 50  0001 C CNN
+F 3 "~" H 4600 5800 50  0001 C CNN
+	1    4600 5800
+	-1   0    0    1
+$EndComp
+$Comp
+L power:VCC #PWR0101
+U 1 1 5C93E913
+P 4600 5550
+F 0 "#PWR0101" H 4600 5400 50  0001 C CNN
+F 1 "VCC" H 4617 5723 50  0000 C CNN
+F 2 "" H 4600 5550 50  0001 C CNN
+F 3 "" H 4600 5550 50  0001 C CNN
+	1    4600 5550
+	1    0    0    -1
+$EndComp
+Wire Wire Line
+	4600 5550 4600 5650
+Wire Wire Line
+	4600 5950 4600 6000
+$Comp
+L Z80-1MSRAM-rescue:GND #PWR0102
+U 1 1 5C96DD5E
+P 4600 6550
+F 0 "#PWR0102" H 4600 6300 50  0001 C CNN
+F 1 "GND" H 4600 6400 50  0000 C CNN
+F 2 "" H 4600 6550 50  0001 C CNN
+F 3 "" H 4600 6550 50  0001 C CNN
+	1    4600 6550
+	1    0    0    -1
+$EndComp
+Wire Wire Line
+	4600 6450 4600 6550
+Text GLabel 5700 6000 2    60   Input ~ 0
+A7
+$Comp
+L Jumper:Jumper_3_Open JP1
+U 1 1 5C985EE7
+P 5300 6000
+F 0 "JP1" H 5300 6224 50  0000 C CNN
+F 1 "A7_Jumper" H 5300 6133 50  0000 C CNN
+F 2 "Connector_PinHeader_2.54mm:PinHeader_1x03_P2.54mm_Vertical" H 5300 6000 50  0001 C CNN
+F 3 "~" H 5300 6000 50  0001 C CNN
+	1    5300 6000
+	1    0    0    -1
+$EndComp
+Wire Wire Line
+	4600 6000 5050 6000
+Connection ~ 4600 6000
+Wire Wire Line
+	4600 6000 4600 6050
+Wire Wire Line
+	5700 6000 5550 6000
+Wire Wire Line
+	5300 6150 5300 6350
+Wire Wire Line
+	5300 6350 5500 6350
+Text Notes 5500 6150 0    60   ~ 0
+0xh-6xh
+Text Notes 4800 6150 0    60   ~ 0
+8xh-Exh
+Text Label 5550 6000 0    60   ~ 0
+A7
+Text Label 3550 6250 0    60   ~ 0
+A7
+$Comp
+L Z80-1MSRAM-rescue:PWR_FLAG #FLG0101
+U 1 1 5CA0C77E
+P 5300 6550
+F 0 "#FLG0101" H 5300 6625 50  0001 C CNN
+F 1 "PWR_FLAG" H 5300 6700 50  0000 C CNN
+F 2 "" H 5300 6550 50  0001 C CNN
+F 3 "" H 5300 6550 50  0001 C CNN
+	1    5300 6550
+	-1   0    0    1
+$EndComp
+Wire Wire Line
+	5300 6550 5300 6350
 Wire Bus Line
 	4850 2700 4850 3250
@@
 Wire Bus Line
 	12400 2600 12400 7350
+Connection ~ 5300 6350
 $EndSCHEMATC

Commit message: REV3 回路図、プリントパターン、ガーバーデータ
Parts:
- added C9: 22p, Capacitor_THT:C_Disc_D3.0mm_W1.6mm_P2.50mm, symbol Device:C
- added JP2: 16k/32k, Connector_PinHeader_2.54mm:PinHeader_1x03_P2.54mm_Vertical, symbol Jumper:Jumper_3_Open
Connections:
- net A14: now also JP2.3 (B); no longer U3.14 (A0)
- net A7: now also C9.2
- net GND: now also JP2.1 (A)
- net at Q1.3 (B), R4.1: now also C9.1
- new net: JP2.2 (C), U3.14 (A0)
Changed lines of the file:
@@
 Sheet 1 1
 Title "SBC8080 128k MEMORY BOARD"
-Date "2019-03-16"
-Rev "2.1"
+Date "2019-09-07"
+Rev "3"
 Comp ""
 Comment1 ""
@@
 	1    0    0    -1
 $EndComp
-Text Label 8400 3300 0    60   ~ 0
+Text Label 8200 2950 2    60   ~ 0
 A14
 Entry Wire Line
-	8300 3200 8400 3300
+	8300 2850 8200 2950
 NoConn ~ 10250 3300
 NoConn ~ 10250 3500
@@
 	8400 5450 8200 5450
 Wire Wire Line
-	8550 3300 8400 3300
-Wire Wire Line
 	8550 3650 8400 3650
 Wire Wire Line
@@
 U 1 1 5C8B2A5C
 P 4000 6250
-F 0 "R4" V 3900 6250 50  0000 C CNN
-F 1 "100k" V 4100 6250 50  0000 C CNN
+F 0 "R4" V 4100 6100 50  0000 C CNN
+F 1 "100k" V 4100 6350 50  0000 C CNN
 F 2 "Resistor_THT:R_Axial_DIN0207_L6.3mm_D2.5mm_P10.16mm_Horizontal" V 4040 6240 50  0001 C CNN
 F 3 "~" H 4000 6250 50  0001 C CNN
@@
 A7
 Wire Wire Line
-	3500 6250 3850 6250
+	3500 6250 3750 6250
 Wire Wire Line
 	4900 3700 5200 3700
@@
 $EndComp
 Wire Wire Line
-	4150 6250 4300 6250
+	4150 6250 4250 6250
 $Comp
 L Device:R_US R5
@@
 	5300 6550 5300 6350
 Connection ~ 5300 6350
+$Comp
+L Device:C C9
+U 1 1 5CA0558F
+P 4000 6000
+F 0 "C9" V 3950 5850 50  0000 C CNN
+F 1 "22p" V 3950 6150 50  0000 C CNN
+F 2 "Capacitor_THT:C_Disc_D3.0mm_W1.6mm_P2.50mm" H 4038 5850 50  0001 C CNN
+F 3 "~" H 4000 6000 50  0001 C CNN
+	1    4000 6000
+	0    1    1    0
+$EndComp
+Wire Wire Line
+	3850 6000 3750 6000
+Wire Wire Line
+	3750 6000 3750 6250
+Connection ~ 3750 6250
+Wire Wire Line
+	3750 6250 3850 6250
+Wire Wire Line
+	4150 6000 4250 6000
+Wire Wire Line
+	4250 6000 4250 6250
+Connection ~ 4250 6250
+Wire Wire Line
+	4250 6250 4300 6250
+$Comp
+L Jumper:Jumper_3_Open JP2
+U 1 1 5D76E08D
+P 7950 3300
+F 0 "JP2" V 8100 3350 50  0000 L CNN
+F 1 "16k/32k" V 8200 3350 50  0000 L CNN
+F 2 "Connector_PinHeader_2.54mm:PinHeader_1x03_P2.54mm_Vertical" H 7950 3300 50  0001 C CNN
+F 3 "~" H 7950 3300 50  0001 C CNN
+	1    7950 3300
+	0    -1   -1   0
+$EndComp
+Wire Wire Line
+	7950 2950 7950 3050
+Wire Wire Line
+	7950 2950 8200 2950
+Wire Wire Line
+	7950 3550 7950 3650
+Wire Wire Line
+	7950 3650 8400 3650
+Connection ~ 8400 3650
+Wire Wire Line
+	8550 3300 8500 3300
+$Comp
+L power:PWR_FLAG #FLG0102
+U 1 1 5D846A51
+P 8500 3350
+F 0 "#FLG0102" H 8500 3425 50  0001 C CNN
+F 1 "PWR_FLAG" H 8500 3523 50  0000 C CNN
+F 2 "" H 8500 3350 50  0001 C CNN
+F 3 "~" H 8500 3350 50  0001 C CNN
+	1    8500 3350
+	-1   0    0    1
+$EndComp
+Wire Wire Line
+	8500 3300 8500 3350
+Connection ~ 8500 3300
+Wire Wire Line
+	8500 3300 8100 3300
+Wire Bus Line
+	4300 2300 4300 5000
 Wire Bus Line
 	4850 2700 4850 3250
-Wire Bus Line
-	4300 2300 4300 5000
 Wire Bus Line
 	2350 2200 14400 2200
@@
 	8300 2700 8300 3800
 Wire Bus Line
-	3400 2300 3400 4000
+	2200 2600 12400 2600
 Wire Bus Line
 	2250 2300 2250 4000
 Wire Bus Line
-	2200 2600 12400 2600
+	3400 2300 3400 4000
+Wire Bus Line
+	2100 2700 2100 5200
 Wire Bus Line
 	3600 2700 3600 5200
 Wire Bus Line
-	2100 2700 2100 5200
-Wire Bus Line
 	14500 2300 14500 6650

Commit message: REV4基板 ガーバーデータ出力
Parts:
- added J3: MSX SLOT, Connector_PinHeader_2.54mm:PinHeader_1x05_P2.54mm_Vertical, symbol Connector_Generic:Conn_01x05
- added JP3: RAMCSJP, Connector_PinHeader_2.54mm:PinHeader_1x03_P2.54mm_Vertical, symbol Jumper:Jumper_3_Open
- added JP4: ROMCSJP, Connector_PinHeader_2.54mm:PinHeader_1x03_P2.54mm_Vertical, symbol Jumper:Jumper_3_Open
Connections:
- new net: JP3.2 (C), U6.30 (CS2)
- new net: JP4.2 (C), U7.20 (CS)
- new net: JP3.3 (B), JP4.3 (B), U1.13
- new net: J3.4 (Pin_4), JP3.1 (A)
- new net: J3.1 (Pin_1), JP4.1 (A)
- no-connect marks 13 -> 16
Changed lines of the file:
@@
 EESchema Schematic File Version 4
 LIBS:Z80-1MSRAM-cache
-EELAYER 26 0
+EELAYER 30 0
 EELAYER END
 $Descr A3 16535 11693
@@
 Sheet 1 1
 Title "SBC8080 128k MEMORY BOARD"
-Date "2019-09-07"
-Rev "3"
+Date "2021-03-22"
+Rev "4"
 Comp ""
 Comment1 ""
@@
 	8400 3150 8550 3150
 Wire Wire Line
-	11250 4950 11250 5400
-Wire Wire Line
 	10400 7900 10400 7550
-Wire Wire Line
-	11250 5400 11850 5400
 Wire Wire Line
 	9600 5350 9750 5350
@@
 	10150 8250 10150 7900
 Connection ~ 10150 7900
-Wire Wire Line
-	11850 5400 11850 5500
 Wire Wire Line
 	11850 5500 12800 5500
@@
 RES
 Wire Wire Line
-	11250 7850 12800 7850
-Connection ~ 11250 5400
-Wire Wire Line
-	11250 5400 11250 7850
-Wire Wire Line
 	7950 7900 8350 7900
 Wire Wire Line
@@
 Wire Wire Line
 	8500 3300 8100 3300
+$Comp
+L Jumper:Jumper_3_Open JP3
+U 1 1 607DD3CF
+P 11250 8500
+F 0 "JP3" V 11296 8587 50  0000 L CNN
+F 1 "RAMCSJP" V 11205 8587 50  0000 L CNN
+F 2 "Connector_PinHeader_2.54mm:PinHeader_1x03_P2.54mm_Vertical" H 11250 8500 50  0001 C CNN
+F 3 "~" H 11250 8500 50  0001 C CNN
+	1    11250 8500
+	0    -1   -1   0
+$EndComp
+$Comp
+L Jumper:Jumper_3_Open JP4
+U 1 1 607DEB6F
+P 12250 8500
+F 0 "JP4" V 12296 8587 50  0000 L CNN
+F 1 "ROMCSJP" V 12205 8587 50  0000 L CNN
+F 2 "Connector_PinHeader_2.54mm:PinHeader_1x03_P2.54mm_Vertical" H 12250 8500 50  0001 C CNN
+F 3 "~" H 12250 8500 50  0001 C CNN
+	1    12250 8500
+	0    -1   -1   0
+$EndComp
+Wire Wire Line
+	12800 7850 12650 7850
+Wire Wire Line
+	12650 7850 12650 8500
+Wire Wire Line
+	12650 8500 12400 8500
+Wire Wire Line
+	11250 4950 11250 8000
+Wire Wire Line
+	11850 5500 11850 8500
+Wire Wire Line
+	11850 8500 11400 8500
+Wire Wire Line
+	11250 8000 12250 8000
+Wire Wire Line
+	12250 8000 12250 8250
+Connection ~ 11250 8000
+Wire Wire Line
+	11250 8000 11250 8250
+Wire Wire Line
+	11250 8750 11250 9400
+Wire Wire Line
+	11250 9400 12850 9400
+Wire Wire Line
+	12250 8750 12250 9100
+$Comp
+L Connector_Generic:Conn_01x05 J3
+U 1 1 608D9FD8
+P 13050 9300
+F 0 "J3" H 13130 9342 50  0000 L CNN
+F 1 "MSX SLOT" H 13130 9251 50  0000 L CNN
+F 2 "Connector_PinHeader_2.54mm:PinHeader_1x05_P2.54mm_Vertical" H 13050 9300 50  0001 C CNN
+F 3 "~" H 13050 9300 50  0001 C CNN
+	1    13050 9300
+	1    0    0    -1
+$EndComp
+Wire Wire Line
+	12250 9100 12850 9100
+NoConn ~ 12850 9200
+NoConn ~ 12850 9300
+NoConn ~ 12850 9500
 Wire Bus Line
 	4300 2300 4300 5000
